File: small-scope.sch (KiCad schematic (older format))
At the start: 41 parts, among them P1 BNC, P2 AREF, SW1 STAT DIS, U1 LM324N

Commit message: initial placement
Parts:
- C5: value 16.9p -> 16p
- C7: value 135p -> 130p
Connections:
- net labels added: 2.5V
Changed lines of the file:
@@
 LIBS:contrib
 LIBS:valves
-LIBS:custom-modules
-LIBS:arduino-modules
-LIBS:arduino_shields
 LIBS:small-scope-cache
 EELAYER 27 0
@@
 $Comp
 L LM324N U1
-U 4 1 540AEA76
+U 3 1 540AEA76
 P 7750 1100
 F 0 "U1" H 7800 1300 60  0000 C CNN
@@
 F 2 "" H 7750 1100 60  0000 C CNN
 F 3 "" H 7750 1100 60  0000 C CNN
-	4    7750 1100
+	3    7750 1100
 	1    0    0    1
 $EndComp
 $Comp
 L LM324N U1
-U 3 1 540AEA83
+U 4 1 540AEA83
 P 9500 2450
 F 0 "U1" H 9550 2650 60  0000 C CNN
@@
 F 2 "" H 9500 2450 60  0000 C CNN
 F 3 "" H 9500 2450 60  0000 C CNN
-	3    9500 2450
+	4    9500 2450
 	1    0    0    -1
 $EndComp
 $Comp
 L LM324N U1
-U 2 1 540AEA89
+U 1 1 540AEA89
 P 5150 6800
 F 0 "U1" H 5200 7000 60  0000 C CNN
@@
 F 2 "" H 5150 6800 60  0000 C CNN
 F 3 "" H 5150 6800 60  0000 C CNN
-	2    5150 6800
+	1    5150 6800
 	1    0    0    1
 $EndComp
 $Comp
 L LM324N U1
-U 1 1 540AEA8F
+U 2 1 540AEA8F
 P 2700 6700
 F 0 "U1" H 2750 6900 60  0000 C CNN
@@
 F 2 "" H 2700 6700 60  0000 C CNN
 F 3 "" H 2700 6700 60  0000 C CNN
-	1    2700 6700
+	2    2700 6700
 	1    0    0    1
 $EndComp
@@
 P 1550 1700
 F 0 "C5" H 1550 1800 40  0000 L CNN
-F 1 "16.9p" H 1556 1615 40  0000 L CNN
+F 1 "16p" H 1556 1615 40  0000 L CNN
 F 2 "~" H 1588 1550 30  0000 C CNN
 F 3 "~" H 1550 1700 60  0000 C CNN
@@
 P 2150 1700
 F 0 "C7" H 2150 1800 40  0000 L CNN
-F 1 "135p" H 2156 1615 40  0000 L CNN
+F 1 "130p" H 2156 1615 40  0000 L CNN
 F 2 "~" H 2188 1550 30  0000 C CNN
 F 3 "~" H 2150 1700 60  0000 C CNN
@@
 F 3 "~" H 1750 5100 30  0000 C CNN
 	1    1750 5100
-	1    0    0    -1
+	1    0    0    1
 $EndComp
 $Comp
@@
 Text Notes 1300 6050 0    60   ~ 0
 LEDS
+Text Label 7450 2350 2    60   ~ 0
+2.5V
 $EndSCHEMATC

Commit message: routing done
Connections:
- wire segments 114 -> 110
- no-connect marks 16 -> 18
Changed lines of the file:
@@
 LIBS:contrib
 LIBS:valves
+LIBS:custom-modules
+LIBS:arduino-modules
+LIBS:arduino_shields
 LIBS:small-scope-cache
 EELAYER 27 0
@@
 	1    3000 2800
 	0    -1   -1   0
-$EndComp
-$Comp
-L GND #PWR010
-U 1 1 540AFB8D
-P 850 3450
-F 0 "#PWR010" H 850 3450 30  0001 C CNN
-F 1 "GND" H 850 3380 30  0001 C CNN
-F 2 "" H 850 3450 60  0000 C CNN
-F 3 "" H 850 3450 60  0000 C CNN
-	1    850  3450
-	0    1    1    0
 $EndComp
 Text Label 1000 3800 2    60   ~ 0
@@
 Wire Wire Line
 	2900 2800 3000 2800
-Wire Wire Line
-	950  3500 1000 3500
-Wire Wire Line
-	950  3400 950  3500
-Wire Wire Line
-	950  3400 1000 3400
-Wire Wire Line
-	950  3450 850  3450
-Connection ~ 950  3450
 Text Label 2900 2900 0    60   ~ 0
 ERR_LED
@@
 Text Label 7450 2350 2    60   ~ 0
 2.5V
+NoConn ~ 1000 3400
+NoConn ~ 1000 3500
 $EndSCHEMATC

Commit message: added AC/DC select and separate DC bias
Parts:
- added C10: 10u/35V, ~, symbol C
- added C11: 10u, ~, symbol CP1
- added JP5: AC/DC, ~, symbol JUMPER3
- added R19: 10k, ~, symbol R
- added RV2: 10k, ~, symbol POT
- JP2: value AC/DC -> DC BIAS
- R3, R5: value 1k -> 10k
Connections:
- net labels added: BIAS, SIG_ACDC
- wire segments 110 -> 126
Other:
- note added: "AC/DC"
- moved on the sheet: C1

Commit message: board rev1
Connections:
- wire segments 126 -> 128
- no-connect marks 18 -> 16
Changed lines of the file:
@@
 LIBS:contrib
 LIBS:valves
-LIBS:custom-modules
-LIBS:arduino-modules
-LIBS:arduino_shields
 LIBS:small-scope-cache
 EELAYER 27 0
@@
 Sheet 1 1
 Title "small scope"
-Date "11 jul 2015"
+Date "13 jul 2015"
 Rev ""
 Comp "Sinister Bureau"
@@
 Text Label 8000 2350 0    60   ~ 0
 BIAS
-NoConn ~ 1000 3400
-NoConn ~ 1000 3500
 $Comp
 L POT RV2
@@
 Wire Wire Line
 	5050 7200 5050 7250
+$Comp
+L GND #PWR?
+U 1 1 55A3B3C7
+P 950 3400
+F 0 "#PWR?" H 950 3400 30  0001 C CNN
+F 1 "GND" H 950 3330 30  0001 C CNN
+F 2 "" H 950 3400 60  0000 C CNN
+F 3 "" H 950 3400 60  0000 C CNN
+	1    950  3400
+	0    1    1    0
+$EndComp
+Wire Wire Line
+	950  3400 1000 3400
+$Comp
+L GND #PWR?
+U 1 1 55A3B494
+P 950 3500
+F 0 "#PWR?" H 950 3500 30  0001 C CNN
+F 1 "GND" H 950 3430 30  0001 C CNN
+F 2 "" H 950 3500 60  0000 C CNN
+F 3 "" H 950 3500 60  0000 C CNN
+	1    950  3500
+	0    1    1    0
+$EndComp
+Wire Wire Line
+	950  3500 1000 3500
 $EndSCHEMATC

Commit message: Fixed reversed power supply on OP amp
Changed lines of the file:
@@
 LIBS:contrib
 LIBS:valves
+LIBS:custom-modules
+LIBS:arduino-modules
+LIBS:arduino_shields
 LIBS:small-scope-cache
 EELAYER 27 0
@@
 Sheet 1 1
 Title "small scope"
-Date "13 jul 2015"
+Date "5 nov 2015"
 Rev ""
 Comp "Sinister Bureau"
@@
 $Comp
 L LM324N U1
-U 3 1 540AEA76
+U 1 1 540AEA76
 P 7750 1100
 F 0 "U1" H 7800 1300 60  0000 C CNN
@@
 F 2 "" H 7750 1100 60  0000 C CNN
 F 3 "" H 7750 1100 60  0000 C CNN
-	3    7750 1100
+	1    7750 1100
 	1    0    0    1
 $EndComp
 $Comp
 L LM324N U1
-U 4 1 540AEA83
+U 2 1 540AEA83
 P 9500 2450
 F 0 "U1" H 9550 2650 60  0000 C CNN
@@
 F 2 "" H 9500 2450 60  0000 C CNN
 F 3 "" H 9500 2450 60  0000 C CNN
-	4    9500 2450
+	2    9500 2450
 	1    0    0    -1
 $EndComp
 $Comp
 L LM324N U1
-U 1 1 540AEA89
+U 3 1 540AEA89
 P 5150 6800
 F 0 "U1" H 5200 7000 60  0000 C CNN
@@
 F 2 "" H 5150 6800 60  0000 C CNN
 F 3 "" H 5150 6800 60  0000 C CNN
-	1    5150 6800
+	3    5150 6800
 	1    0    0    1
 $EndComp
 $Comp
 L LM324N U1
-U 2 1 540AEA8F
+U 4 1 540AEA8F
 P 2700 6700
 F 0 "U1" H 2750 6900 60  0000 C CNN
@@
 F 2 "" H 2700 6700 60  0000 C CNN
 F 3 "" H 2700 6700 60  0000 C CNN
-	2    2700 6700
+	4    2700 6700
 	1    0    0    1
 $EndComp
@@
 L GND #PWR07
 U 1 1 540AF97B
-P 5050 7250
-F 0 "#PWR07" H 5050 7250 30  0001 C CNN
-F 1 "GND" H 5050 7180 30  0001 C CNN
-F 2 "" H 5050 7250 60  0000 C CNN
-F 3 "" H 5050 7250 60  0000 C CNN
-	1    5050 7250
-	1    0    0    -1
+P 5050 6350
+F 0 "#PWR07" H 5050 6350 30  0001 C CNN
+F 1 "GND" H 5050 6280 30  0001 C CNN
+F 2 "" H 5050 6350 60  0000 C CNN
+F 3 "" H 5050 6350 60  0000 C CNN
+	1    5050 6350
+	-1   0    0    1
 $EndComp
 $Comp
@@
 L VDD #PWR019
 U 1 1 555A0D50
-P 5050 6350
-F 0 "#PWR019" H 5050 6450 30  0001 C CNN
-F 1 "VDD" H 5050 6460 30  0000 C CNN
-F 2 "" H 5050 6350 60  0000 C CNN
-F 3 "" H 5050 6350 60  0000 C CNN
-	1    5050 6350
-	1    0    0    -1
+P 5050 7250
+F 0 "#PWR019" H 5050 7350 30  0001 C CNN
+F 1 "VDD" H 5050 7360 30  0000 C CNN
+F 2 "" H 5050 7250 60  0000 C CNN
+F 3 "" H 5050 7250 60  0000 C CNN
+	1    5050 7250
+	-1   0    0    1
 $EndComp
 $Comp
@@
 	5050 7200 5050 7250
 $Comp
-L GND #PWR?
+L GND #PWR030
 U 1 1 55A3B3C7
 P 950 3400
-F 0 "#PWR?" H 950 3400 30  0001 C CNN
+F 0 "#PWR030" H 950 3400 30  0001 C CNN
 F 1 "GND" H 950 3330 30  0001 C CNN
 F 2 "" H 950 3400 60  0000 C CNN
@@
 	950  3400 1000 3400
 $Comp
-L GND #PWR?
+L GND #PWR031
 U 1 1 55A3B494
 P 950 3500
-F 0 "#PWR?" H 950 3500 30  0001 C CNN
+F 0 "#PWR031" H 950 3500 30  0001 C CNN
 F 1 "GND" H 950 3430 30  0001 C CNN
 F 2 "" H 950 3500 60  0000 C CNN
